File: Hardware/EdgeBoard/KiCad/MaD_Edge.kicad_pcb (KiCad board)
At the start: 4 copper layers, 144.1 x 93.3 mm, 280 parts, among them IC1 ISO6742DWR, IC10 NSI50010YT1G, IC11 NSI50010YT1G, IC12 NSI50010YT1G, IC13 NSI50010YT1G, IC14 ISO6741DWR, IC15 ISO6721BDR, IC16 ISO6740FDWR, IC2 ISO6742DWR, IC3 UCC12040DVER, IC4 UCC12040DVER, IC5 ISO6731DWR, IC6 NSI50010YT1G, IC7 NSI50010YT1G, IC8 NSI50010YT1G, IC9 NSI50010YT1G, J1 Debug, J10 ChargePump, J11 ESDUpper, J12 ESDLower, J13 ESDActive, J14 ENDUpper, J15 ENDLower, J16 Door, J17 GPI_3, J18 GPI_4, J19 NavKey, J2 Main_Power, J20 Encoder, J21 ServoCtrl, J22 GPIO_EXT_1, J23 ServoSerial, J24 GPIO_EXT_2, J3 P2_EDGE_MODULE_SOCKET, J4 RPI, J5 GPO_2, J6 GPO_1, J7 GPI_2, J8 GPI_1, J9 Force, Q1 NPN, SW1 RESET, U1 XL1509-5V, U10 SN74LVC1G14DBV, U11 SN74LVC1G14DBV, U12 SN74LVC1G14DBV, U13 SN74LVC1G14DBV, U14 SN74LVC1G14DBV, U15 SN74LVC1G14DBV, U16 SN74LVC1G14DBV, U17 SN74LVC1G14DBV, U18 SN74LVC1G14DBV, U19 SN74LVC1G14DBV, U2 XL1509-3.3V, U21 SN74LVC1G14DBV, U22 SN74LVC1G14DBV, U24 AM26LS31CD, U25 AM26LV32xD, U27 SN74LVC1G14DBV, U28 SN74LVC1G14DBV, U29 SN74LVC1G14DBV, U3 APM4953, U30 SN74LVC1G14DBV, U31 SN74LVC1G14DBV, U32 SN74LVC1G14DBV, U33 SN74LVC1G14DBV, U34 SN74LVC1G14DBV, U4 6N137, U5 VO2631, U6 VO2631, U7 VO2631, U8 VO2631, U9 SN74LVC1G14DBV

Commit message: DS2 and MaDEdge updates
Parts:
- J4: value RPI -> 436500321; footprint Connector_Molex:Molex_Micro-Fit_3.0_43045-0618_2x03-1MP_P3.00mm_Vertical -> Connector_Molex:Molex_Micro-Fit_3.0_43045-0615_2x03_P3.00mm_Vertical
- moved kibuzzard-6474D12A 15.6 mm to (87.5, 199.6)
- moved kibuzzard-6474D10F 15.4 mm to (103.0, 199.6)
- moved kibuzzard-647770D0 12.4 mm to (1.00, 157.0)
- moved kibuzzard-6477707F 12.4 mm to (13.0, 160.5)
- moved kibuzzard-64777917 3.23 mm to (123.0, 120.0)
- moved kibuzzard-64777922 2.80 mm to (120.0, 120.0)
Connections:
- IC11 pad 2: /MaD_Edge_Sheet2/IEND_U+ -> /MaD_Edge_Sheet2/IDOOR+
- IC2 pad 12: /MaD_Edge_Sheet2/RPI_TX -> /MaD_Edge_Sheet2/RPI_RX
- IC2 pad 14: /MaD_Edge_Sheet2/RPI_RX -> /MaD_Edge_Sheet2/RPI_TX
- IC5 pad 3: /MaD_Edge_Sheet2/IFG_TX -> /MaD_Edge_Sheet2/IFG_RX
- IC5 pad 5: /MaD_Edge_Sheet2/IFG_RX -> /MaD_Edge_Sheet2/IFG_TX
- IC9 pad 2: /MaD_Edge_Sheet2/IDOOR+ -> /MaD_Edge_Sheet2/IEND_U+
- J14 pad 1: /MaD_Edge_Sheet2/IEND_U- -> /MaD_Edge_Sheet2/IDOOR-
- J14 pad 2: /MaD_Edge_Sheet2/IEND_U+ -> /MaD_Edge_Sheet2/IDOOR+
- J16 pad 1: /MaD_Edge_Sheet2/IDOOR- -> /MaD_Edge_Sheet2/IEND_U-
- J16 pad 2: /MaD_Edge_Sheet2/IDOOR+ -> /MaD_Edge_Sheet2/IEND_U+
- J4 pad 2: /MaD_Edge_Sheet2/RPI_RX -> /MaD_Edge_Sheet2/RPI_TX
- J4 pad 3: /MaD_Edge_Sheet2/RPI_TX -> /MaD_Edge_Sheet2/RPI_RX
- J9 pad 2: /MaD_Edge_Sheet2/IFG_TX -> /MaD_Edge_Sheet2/IFG_RX
- J9 pad 4: /MaD_Edge_Sheet2/IFG_RX -> /MaD_Edge_Sheet2/IFG_TX
- U6 pad 3: /MaD_Edge_Sheet2/IDOOR- -> /MaD_Edge_Sheet2/IEND_U-
- U7 pad 3: /MaD_Edge_Sheet2/IEND_U- -> /MaD_Edge_Sheet2/IDOOR-
Routing:
- net /MaD_Edge_Sheet2/IFG_TX: track 8.46 -> 18.1 mm
- net /MaD_Edge_Sheet2/IFG_RX: track 18.1 -> 8.46 mm
- net /MaD_Edge_Sheet2/RPI_TX: track 16.8 -> 13.7 mm
- net /MaD_Edge_Sheet2/RPI_RX: track 13.7 -> 16.8 mm
- net /MaD_Edge_Sheet2/IEND_U-: track 11.1 -> 10.3 mm
- net /MaD_Edge_Sheet2/IDOOR-: track 10.3 -> 11.1 mm
- net /MaD_Edge_Sheet2/IEND_U+: track 6.36 -> 5.77 mm
- net /MaD_Edge_Sheet2/IDOOR+: track 5.77 -> 6.36 mm
Other:
- board text added: "E_SW"
- board text added: "SHIELD"
- board text removed: "E_EN"
