File: Hardware/EdgeBoard/KiCad/MaD_Edge.kicad_pcb (KiCad board)
At the start: 4 copper layers, 144.1 x 93.3 mm, 280 parts, among them IC1 ISO6742DWR, IC10 NSI50010YT1G, IC11 NSI50010YT1G, IC12 NSI50010YT1G, IC13 NSI50010YT1G, IC14 ISO6741DWR, IC15 ISO6721BDR, IC16 ISO6740FDWR, IC2 ISO6742DWR, IC3 UCC12040DVER, IC4 UCC12040DVER, IC5 ISO6731DWR, IC6 NSI50010YT1G, IC7 NSI50010YT1G, IC8 NSI50010YT1G, IC9 NSI50010YT1G, J1 Debug, J10 ChargePump, J11 ESDUpper, J12 ESDLower, J13 ESDActive, J14 ENDUpper, J15 ENDLower, J16 Door, J17 GPI_3, J18 GPI_4, J19 NavKey, J2 Main_Power, J20 Encoder, J21 ServoCtrl, J22 GPIO_EXT_1, J23 ServoSerial, J24 GPIO_EXT_2, J3 P2_EDGE_MODULE_SOCKET, J4 436500321, J5 GPO_2, J6 GPO_1, J7 GPI_2, J8 GPI_1, J9 Force, Q1 NPN, SW1 RESET, U1 XL1509-5V, U10 SN74LVC1G14DBV, U11 SN74LVC1G14DBV, U12 SN74LVC1G14DBV, U13 SN74LVC1G14DBV, U14 SN74LVC1G14DBV, U15 SN74LVC1G14DBV, U16 SN74LVC1G14DBV, U17 SN74LVC1G14DBV, U18 SN74LVC1G14DBV, U19 SN74LVC1G14DBV, U2 XL1509-3.3V, U21 SN74LVC1G14DBV, U22 SN74LVC1G14DBV, U24 AM26LS31CD, U25 AM26LV32xD, U27 SN74LVC1G14DBV, U28 SN74LVC1G14DBV, U29 SN74LVC1G14DBV, U3 APM4953, U30 SN74LVC1G14DBV, U31 SN74LVC1G14DBV, U32 SN74LVC1G14DBV, U33 SN74LVC1G14DBV, U34 SN74LVC1G14DBV, U4 6N137, U5 VO2631, U6 VO2631, U7 VO2631, U8 VO2631, U9 SN74LVC1G14DBV

Commit message: fix(hardware): update U25's PCB fields to AM26LV32IDR to match the schematic
Fixes #250

## What changed

#244 corrected U25 in the Edge schematic but left the PCB footprint behind. This updates the two U25 footprint properties in `Hardware/EdgeBoard/KiCad/MaD_Edge.kicad_pcb` (footprint uuid `c6927fc4-b34f-4fca-b52d-65d4bd70e1b2`) to match `MaD_Edge_Sheet3.kicad_sch`:

- `Value`: `AM26LV32xD` → `AM26LV32IDR`
- `Manufacturer_Part_Number`: `AM26LS32CD` → `AM26LV32IDR`

The text was edited by hand rather than re-saved through KiCad, so the file stays byte-identical everywhere else and remains a KiCad 9 board (`version 20241229`, `generator_version "9.0"`). U24 (`AM26LS31CD`, the driver) is untouched. No Vibes ledger change.

## How to verify

- `git diff origin/main -- Hardware/` shows exactly two changed lines (61458 and 61506), both inside footprint U25.
- `rg -n "AM26LS32CD" Hardware/EdgeBoard` finds nothing.
- `rg -n 'generator_version' Hardware/EdgeBoard/KiCad/MaD_Edge.kicad_pcb` still shows `"9.0"`.
- The `build-hardware (EdgeBoard)` CI job (KiBot, KiCad 9) passes; in its BOM artifact U25 is listed as AM26LV32IDR.

## Reviewer notes

The F.Fab `Value` text on U25 now renders as `AM26LV32IDR` (one character longer than before); its placement and size are unchanged.
Parts:
- U25: value AM26LV32xD -> AM26LV32IDR
Changed lines of the file:
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@@
 			)
 		)
-		(property "Value" "AM26LV32xD"
+		(property "Value" "AM26LV32IDR"
 			(at 0 5.9 90)
 			(layer "F.Fab")
@@
 			)
 		)
-		(property "Manufacturer_Part_Number" "AM26LS32CD"
+		(property "Manufacturer_Part_Number" "AM26LV32IDR"
 			(at 0 0 90)
 			(unlocked yes)
