File: Hardware/EdgeBoard/KiCad/MaD_Edge.kicad_pcb (KiCad board)
At the start: 4 copper layers, 144.1 x 93.3 mm, 280 parts, among them IC1 ISO6742DWR, IC10 NSI50010YT1G, IC11 NSI50010YT1G, IC12 NSI50010YT1G, IC13 NSI50010YT1G, IC14 ISO6741DWR, IC15 ISO6721BDR, IC16 ISO6740FDWR, IC2 ISO6742DWR, IC3 UCC12040DVER, IC4 UCC12040DVER, IC5 ISO6731DWR, IC6 NSI50010YT1G, IC7 NSI50010YT1G, IC8 NSI50010YT1G, IC9 NSI50010YT1G, J1 Debug, J10 ChargePump, J11 ESDUpper, J12 ESDLower, J13 ESDActive, J14 ENDUpper, J15 ENDLower, J16 Door, J17 GPI_3, J18 GPI_4, J19 NavKey, J2 Main_Power, J20 Encoder, J21 ServoCtrl, J22 GPIO_EXT_1, J23 ServoSerial, J24 GPIO_EXT_2, J3 P2_EDGE_MODULE_SOCKET, J4 436500321, J5 GPO_2, J6 GPO_1, J7 GPI_2, J8 GPI_1, J9 Force, Q1 NPN, SW1 RESET, U1 XL1509-5V, U10 SN74LVC1G14DBV, U11 SN74LVC1G14DBV, U12 SN74LVC1G14DBV, U13 SN74LVC1G14DBV, U14 SN74LVC1G14DBV, U15 SN74LVC1G14DBV, U16 SN74LVC1G14DBV, U17 SN74LVC1G14DBV, U18 SN74LVC1G14DBV, U19 SN74LVC1G14DBV, U2 XL1509-3.3V, U21 SN74LVC1G14DBV, U22 SN74LVC1G14DBV, U24 AM26LS31CD, U25 AM26LV32IDR, U27 SN74LVC1G14DBV, U28 SN74LVC1G14DBV, U29 SN74LVC1G14DBV, U3 APM4953, U30 SN74LVC1G14DBV, U31 SN74LVC1G14DBV, U32 SN74LVC1G14DBV, U33 SN74LVC1G14DBV, U34 SN74LVC1G14DBV, U4 6N137, U5 VO2631, U6 VO2631, U7 VO2631, U8 VO2631, U9 SN74LVC1G14DBV

Commit message: fix(hardware): servo enable off at power-up: IC14 ISO7741FDWR and a P6 pull-down
Finding SRV-F6. Nothing pulls P6 (servo enable request), and the fitted
non-F IC14 outputs high from an open or unpowered input, so the drive
enable is on through reset, boot and flashing.

- IC14 becomes ISO7741FDWR (LCSC C485810): same pinout (TI SLLSEP4K
  Table 4-1 p.5); with the F suffix an open input or an unpowered side 1
  gives a low output (Table 7-2 p.29). Value, MPN, LCSC and notes updated.
- R39, 10 k (0603WAF1002T5E, C25804) from P6 to GND. On the PCB it sits
  by IC14 and joins the P6 trace at U29 through two 0.6 mm vias and B.Cu.
- STEP/DIR (P8/P7) now also rest low when undriven.

Co-Authored-By: Claude Opus 5.5 <noreply@anthropic.com>
Parts:
- added R39: 10K, Resistor_SMD:R_0603_1608Metric, F.Cu at (31.2, 171.5)
- IC14: value ISO6741DWR -> ISO7741FDWR
Routing:
- net P6: track 25.6 -> 36.0 mm, vias 0 -> 2
- net GND: track 333.3 -> 334.9 mm

Commit message: fix(hardware): Q1 drawn and laid out as the fitted SOT-23 MMBT3904
Finding SRV-F8-Q1. Q1 used the TO-92 2N3904 symbol (1 E, 2 B, 3 C) but
the part fitted is a SOT-23 MMBT3904 (1 B, 2 E, 3 C; JSCJ datasheet,
LCSC C20526, p.1), so JP1's open-collector position could never enable
the drive.

- Symbol Transistor_BJT:MMBT3904, footprint Package_TO_SOT_SMD:SOT-23.
- PCB: Q1 rotated -90 so base faces R24; base to R24, emitter to a new
  EN_GND via, collector to JP1 pin 3. The old emitter trace and via go.

Co-Authored-By: Claude Opus 5.5 <noreply@anthropic.com>
Parts:
- Q1: value NPN -> MMBT3904; footprint Package_TO_SOT_SMD:TSOT-23 -> Package_TO_SOT_SMD:SOT-23
- turned Q1 to -90 degrees
Connections:
- Q1 pad 1: /MaD_Edge_Sheet3/EN_GND -> Net-(Q1-B)
- Q1 pad 2: Net-(Q1-B) -> /MaD_Edge_Sheet3/EN_GND

Commit message: fix(hardware): U25 AM26C32IDR (5 V receiver) with its own 0.1 uF
Finding ENC-F3. U25 (AM26LV32IDR, 3.0-3.6 V, TI SLLS202H 6.3) runs from
the 5 V SC_5V rail.

- U25 becomes AM26C32IDR (LCSC C36693): pin-identical (TI SLLS104M
  Table 4-1 p.3), VCC 4.5-5.5 V (5.3 p.4), VOH >= 3.8 V at -6 mA (5.6
  p.5), above IC16's 0.7 x VCC1 input threshold. KiCad has no AM26C32
  symbol; the AM26LV32xD symbol stays.
- C30, 0.1 uF 0402 (CL05B104KO5NNNC, C1525) from U25.16 to EN_GND,
  beside the pin. 0402 is the size that fits between JP2 and U25.

Co-Authored-By: Claude Opus 5.5 <noreply@anthropic.com>
Parts:
- added C30: 0.1uF, Capacitor_SMD:C_0402_1005Metric, F.Cu at (51.3, 189.4)
- U25: value AM26LV32IDR -> AM26C32IDR
Routing:
- net /MaD_Edge_Sheet3/EN_GND: track 36.6 -> 38.6 mm
- net /MaD_Edge_Sheet3/SC_5V: track 16.6 -> 18.0 mm

Commit message: fix(hardware): U25 always enabled; Z+/Z- on receiver 4; JP4 removed
Finding ENC-F5. U25's enables (G pin 4, ~G pin 12) were wired to J20's
Z+/Z-, so they needed a shunt on JP4 that the BOM did not have, and
receiver 4 was unused.

- G to SC_5V, ~G to EN_GND (SLLS104M Table 7-1 p.9): always enabled.
  The two under-body vias are re-netted to the In2/In1 planes.
- Z+/Z- (J20.7/.8) to 4A/4B (pins 14/15); 4Y reaches P12 through IC16
  channel D. New B.Cu routes and two vias under U25, clear of the
  IC16-INA/INB traces that cross the body.
- JP4 deleted (schematic and PCB).

Co-Authored-By: Claude Opus 5.5 <noreply@anthropic.com>
Parts:
- removed JP4: Z_GND, Connector_PinHeader_2.54mm:PinHeader_1x02_P2.54mm_Vertical
Connections:
- U25 pad 12: /MaD_Edge_Sheet3/Z- -> /MaD_Edge_Sheet3/EN_GND
- U25 pad 14: unconnected-(U25-4A-Pad14) -> /MaD_Edge_Sheet3/Z+
- U25 pad 15: unconnected-(U25-4B-Pad15) -> /MaD_Edge_Sheet3/Z-
- U25 pad 4: /MaD_Edge_Sheet3/Z+ -> /MaD_Edge_Sheet3/SC_5V
Routing:
- net /MaD_Edge_Sheet3/Z-: track 30.3 -> 26.2 mm
- net /MaD_Edge_Sheet3/SC_5V: track 18.0 -> 19.7 mm, vias 7 -> 8
- net /MaD_Edge_Sheet3/Z+: track 19.8 -> 21.5 mm
- net /MaD_Edge_Sheet3/EN_GND: track 38.6 -> 40.4 mm, vias 11 -> 12
