File: Hardware/EdgeBoard/KiCad/MaD_Edge.kicad_pcb (KiCad board)
At the start: 4 copper layers, 144.1 x 93.3 mm, 280 parts, among them IC1 ISO6742DWR, IC10 NSI50010YT1G, IC11 NSI50010YT1G, IC12 NSI50010YT1G, IC13 NSI50010YT1G, IC14 ISO6741DWR, IC15 ISO6721BDR, IC16 ISO6740FDWR, IC2 ISO6742DWR, IC3 UCC12040DVER, IC4 UCC12040DVER, IC5 ISO6731DWR, IC6 NSI50010YT1G, IC7 NSI50010YT1G, IC8 NSI50010YT1G, IC9 NSI50010YT1G, J1 Debug, J10 ChargePump, J11 ESDUpper, J12 ESDLower, J13 ESDActive, J14 ENDUpper, J15 ENDLower, J16 Door, J17 GPI_3, J18 GPI_4, J19 NavKey, J2 Main_Power, J20 Encoder, J21 ServoCtrl, J22 GPIO_EXT_1, J23 ServoSerial, J24 GPIO_EXT_2, J3 P2_EDGE_MODULE_SOCKET, J4 436500321, J5 GPO_2, J6 GPO_1, J7 GPI_2, J8 GPI_1, J9 Force, Q1 NPN, SW1 RESET, U1 XL1509-5V, U10 SN74LVC1G14DBV, U11 SN74LVC1G14DBV, U12 SN74LVC1G14DBV, U13 SN74LVC1G14DBV, U14 SN74LVC1G14DBV, U15 SN74LVC1G14DBV, U16 SN74LVC1G14DBV, U17 SN74LVC1G14DBV, U18 SN74LVC1G14DBV, U19 SN74LVC1G14DBV, U2 XL1509-3.3V, U21 SN74LVC1G14DBV, U22 SN74LVC1G14DBV, U24 AM26LS31CD, U25 AM26LV32IDR, U27 SN74LVC1G14DBV, U28 SN74LVC1G14DBV, U29 SN74LVC1G14DBV, U3 APM4953, U30 SN74LVC1G14DBV, U31 SN74LVC1G14DBV, U32 SN74LVC1G14DBV, U33 SN74LVC1G14DBV, U34 SN74LVC1G14DBV, U4 6N137, U5 VO2631, U6 VO2631, U7 VO2631, U8 VO2631, U9 SN74LVC1G14DBV

Commit message: fix(hardware): ground IC14's drive side (GND2) to EN_GND on the Edge board
IC14 (ISO6741DWR, the servo STEP/DIR/ENA/SRDY isolator) had its GND2 pins
9 and 15 on an isolated net, Net-(IC14-GND2_1), with only C26: no EN_GND
in the schematic and no connection to the EN_GND pour in the layout. As
drawn, the drive-side half of the isolator had no ground return.

Schematic: an EN_GND label on GND2's wire puts pins 9 and 15 and C26.2 on
EN_GND with J21.8 and the rest of the drive side.

Layout: the 3 pads, 10 traces and 2 vias of the old net move to EN_GND.
Both vias already sit inside the In1.Cu EN_GND pour, which is refilled so
it now joins them. The file stays in KiCad 9 format for KiBot; the new
fill was computed by KiCad 10 and matches a fresh refill exactly.

DRC: 0 unconnected; net_conflict 4 -> 1; schematic parity 105 -> 102;
other violations unchanged. ERC errors unchanged (9, all pre-existing).

Co-Authored-By: Claude Opus 5.5 <noreply@anthropic.com>
Connections:
- C26 pad 2: Net-(IC14-GND2_1) -> /MaD_Edge_Sheet3/EN_GND
- IC14 pad 15: Net-(IC14-GND2_1) -> /MaD_Edge_Sheet3/EN_GND
- IC14 pad 9: Net-(IC14-GND2_1) -> /MaD_Edge_Sheet3/EN_GND
Routing:
- net /MaD_Edge_Sheet3/EN_GND: track 22.9 -> 37.1 mm, vias 9 -> 11
- net Net-(IC14-GND2_1): track 14.2 -> 0.00 mm, vias 2 -> 0
Changed lines of the file:
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@@
 			(size 0.65 1.95)
 			(layers "F.Cu" "F.Mask" "F.Paste")
-			(net 1 "Net-(IC14-GND2_1)")
+			(net 227 "/MaD_Edge_Sheet3/EN_GND")
 			(pinfunction "GND2_1")
 			(pintype "passive")
@@
 			(size 0.65 1.95)
 			(layers "F.Cu" "F.Mask" "F.Paste")
-			(net 1 "Net-(IC14-GND2_1)")
+			(net 227 "/MaD_Edge_Sheet3/EN_GND")
 			(pinfunction "GND2_2")
 			(pintype "passive")
@@
 			(layers "F.Cu" "F.Mask" "F.Paste")
 			(roundrect_rratio 0.25)
-			(net 1 "Net-(IC14-GND2_1)")
+			(net 227 "/MaD_Edge_Sheet3/EN_GND")
 			(pintype "passive")
 		)
@@
 		(width 0.25)
 		(layer "F.Cu")
-		(net 1)
+		(net 227)
 	)
 	(segment
@@
 		(width 0.25)
 		(layer "F.Cu")
-		(net 1)
+		(net 227)
 	)
 	(segment
@@
 		(width 0.25)
 		(layer "F.Cu")
-		(net 1)
+		(net 227)
 	)
 	(segment
@@
 		(width 0.25)
 		(layer "F.Cu")
-		(net 1)
+		(net 227)
 	)
 	(segment
@@
 		(width 0.25)
 		(layer "F.Cu")
-		(net 1)
+		(net 227)
 	)
 	(segment
@@
 		(width 0.25)
 		(layer "F.Cu")
-		(net 1)
+		(net 227)
 	)
 	(via
@@
 		(drill 0.4)
 		(layers "F.Cu" "B.Cu")
-		(net 1)
+		(net 227)
 	)
 	(via
@@
 		(drill 0.4)
 		(layers "F.Cu" "B.Cu")
-		(net 1)
+		(net 227)
 	)
 	(segment
@@
 		(width 0.25)
 		(layer "B.Cu")
-		(net 1)
+		(net 227)
 	)
 	(segment
@@
 		(width 0.25)
 		(layer "B.Cu")
-		(net 1)
+		(net 227)
 	)
 	(segment
@@
 		(width 0.25)
 		(layer "B.Cu")
-		(net 1)
+		(net 227)
 	)
 	(segment
@@
 		(width 0.25)
 		(layer "B.Cu")
-		(net 1)
+		(net 227)
 	)
 	(segment

Commit message: Edge carrier revision: fixes from the SIL hardware findings (#309)
* fix(hardware): servo enable off at power-up: IC14 ISO7741FDWR and a P6 pull-down

Finding SRV-F6. Nothing pulls P6 (servo enable request), and the fitted
non-F IC14 outputs high from an open or unpowered input, so the drive
enable is on through reset, boot and flashing.

- IC14 becomes ISO7741FDWR (LCSC C485810): same pinout (TI SLLSEP4K
  Table 4-1 p.5); with the F suffix an open input or an unpowered side 1
  gives a low output (Table 7-2 p.29). Value, MPN, LCSC and notes updated.
- R39, 10 k (0603WAF1002T5E, C25804) from P6 to GND. On the PCB it sits
  by IC14 and joins the P6 trace at U29 through two 0.6 mm vias and B.Cu.
- STEP/DIR (P8/P7) now also rest low when undriven.

Co-Authored-By: Claude Opus 5.5 <noreply@anthropic.com>

* fix(hardware): Q1 drawn and laid out as the fitted SOT-23 MMBT3904

Finding SRV-F8-Q1. Q1 used the TO-92 2N3904 symbol (1 E, 2 B, 3 C) but
the part fitted is a SOT-23 MMBT3904 (1 B, 2 E, 3 C; JSCJ datasheet,
LCSC C20526, p.1), so JP1's open-collector position could never enable
the drive.

- Symbol Transistor_BJT:MMBT3904, footprint Package_TO_SOT_SMD:SOT-23.
- PCB: Q1 rotated -90 so base faces R24; base to R24, emitter to a new
  EN_GND via, collector to JP1 pin 3. The old emitter trace and via go.

Co-Authored-By: Claude Opus 5.5 <noreply@anthropic.com>

* fix(hardware): U25 AM26C32IDR (5 V receiver) with its own 0.1 uF

Finding ENC-F3. U25 (AM26LV32IDR, 3.0-3.6 V, TI SLLS202H 6.3) runs from
the 5 V SC_5V rail.

- U25 becomes AM26C32IDR (LCSC C36693): pin-identical (TI SLLS104M
  Table 4-1 p.3), VCC 4.5-5.5 V (5.3 p.4), VOH >= 3.8 V at -6 mA (5.6
  p.5), above IC16's 0.7 x VCC1 input threshold. KiCad has no AM26C32
  symbol; the AM26LV32xD symbol stays.
- C30, 0.1 uF 0402 (CL05B104KO5NNNC, C1525) from U25.16 to EN_GND,
  beside the pin. 0402 is the size that fits between JP2 and U25.

Co-Authored-By: Claude Opus 5.5 <noreply@anthropic.com>

* fix(hardware): U25 alw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
Parts:
- removed JP4: Z_GND, Connector_PinHeader_2.54mm:PinHeader_1x02_P2.54mm_Vertical
- removed kibuzzard-6477790B: G***, kibuzzard-6477790B
- added C30: 0.1uF, Capacitor_SMD:C_0402_1005Metric, F.Cu at (51.3, 189.4)
- added C31: 0.1uF, Capacitor_SMD:C_0603_1608Metric, F.Cu at (44.8, 185.0)
- added F1: 0.2A/30V, Fuse:Fuse_1206_3216Metric, F.Cu at (38.6, 204.6)
- added J25: ENC_PWR, Connector_PinHeader_2.54mm:PinHeader_1x03_P2.54mm_Vertical, F.Cu at (36.1, 208.3)
- added JP6: Z_REF, Connector_PinHeader_2.54mm:PinHeader_1x02_P2.54mm_Vertical, F.Cu at (49.0, 194.1)
- added R39: 10K, Resistor_SMD:R_0603_1608Metric, F.Cu at (31.2, 171.5)
- added R40: 2.2K, Resistor_SMD:R_0603_1608Metric, F.Cu at (38.5, 201.8)
- added R41: 2.2K, Resistor_SMD:R_0603_1608Metric, F.Cu at (38.5, 198.2)
- added R42: 2.2K, Resistor_SMD:R_0603_1608Metric, F.Cu at (38.5, 200.0)
- added R43: 2.2K, Resistor_SMD:R_0603_1608Metric, F.Cu at (41.6, 185.0)
- added R44: 2.2K, Resistor_SMD:R_0603_1608Metric, F.Cu at (43.2, 185.0)
- IC14: value ISO6741DWR -> ISO7741FDWR
- J4: footprint Connector_Molex:Molex_Micro-Fit_3.0_43045-0615_2x03_P3.00mm_Vertical -> Connector_Molex:Molex_Micro-Fit_3.0_43045-0618_2x03-1MP_P3.00mm_Vertical
- JP2: value A_GND -> A_REF
- JP3: value B_GND -> B_REF
- JP5: value ZI_GND -> ZI_REF
- Q1: value NPN -> MMBT3904; footprint Package_TO_SOT_SMD:TSOT-23 -> Package_TO_SOT_SMD:SOT-23
- R24: value 43K -> 4.7K
- U25: value AM26LV32IDR -> AM26C32IDR
- moved kibuzzard-6474D3A4 2.20 mm to (45.5, 182.1)
- moved kibuzzard-647774DE 0.25 mm to (19.7, 191.8)
- turned Q1 to -90 degrees
Connections:
- net /MaD_Edge_Sheet2/RPI_5V renamed /MaD_Edge_Sheet2/RPI_3V3
- IC2 pad 3: P55 -> P32
- IC2 pad 4: P54 -> P31
- IC2 pad 5: P53 -> P30
- IC2 pad 6: P52 -> P29
- JP2 pad 2: /MaD_Edge_Sheet3/EN_GND -> /MaD_Edge_Sheet3/ENC_REF
- JP3 pad 2: /MaD_Edge_Sheet3/EN_GND -> /MaD_Edge_Sheet3/ENC_REF
- JP5 pad 2: /MaD_Edge_Sheet3/EN_GND -> /MaD_Edge_Sheet3/ENC_REF
- Q1 pad 1: /MaD_Edge_Sheet3/EN_GND -> Net-(Q1-B)
- Q1 pad 2: Net-(Q1-B) -> /MaD_Edge_Sheet3/EN_GND
- U25 pad 12: /MaD_Edge_Sheet3/Z- -> /MaD_Edge_Sheet3/EN_GND
- U25 pad 14: unconnected-(U25-4A-Pad14) -> /MaD_Edge_Sheet3/Z+
- U25 pad 15: unconnected-(U25-4B-Pad15) -> /MaD_Edge_Sheet3/Z-
- U25 pad 4: /MaD_Edge_Sheet3/Z+ -> /MaD_Edge_Sheet3/SC_5V
Routing:
- net P32: track 3.09 -> 56.9 mm, vias 0 -> 1
- net P29: track 0.00 -> 53.8 mm, vias 0 -> 2
- net P30: track 0.00 -> 53.2 mm, vias 0 -> 2
- net P31: track 0.00 -> 52.6 mm, vias 0 -> 2
- net P55: track 49.3 -> 0.00 mm
- net P54: track 47.5 -> 0.00 mm
- net P52: track 46.9 -> 0.00 mm
- net P53: track 45.9 -> 0.00 mm
- net /MaD_Edge_Sheet3/ENC_REF: track 0.00 -> 21.8 mm, vias 0 -> 1
- net /MaD_Edge_Sheet3/Z+: track 19.8 -> 39.1 mm, vias 2 -> 3
- net /MaD_Edge_Sheet3/B+: track 8.57 -> 23.6 mm, vias 0 -> 2
- net /MaD_Edge_Sheet3/A+: track 11.7 -> 22.9 mm, vias 0 -> 2
- net P6: track 25.6 -> 36.0 mm, vias 0 -> 2
- net /MaD_Edge_Sheet3/SC_5V: track 16.6 -> 25.5 mm, vias 7 -> 10
- net /MaD_Edge_Sheet3/EN_GND: track 37.1 -> 43.8 mm, vias 11 -> 14
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- added copper zone on B.Cu, net Net-(IC10-K)
- added copper zone on F.Cu, net Net-(IC10-K)
- added copper zone on In1.Cu, net Net-(IC10-K)
- added copper zone on In2.Cu, net Net-(IC10-K)
- added copper zone on B.Cu, net Net-(IC11-K)
- added copper zone on F.Cu, net Net-(IC11-K)
- added copper zone on In1.Cu, net Net-(IC11-K)
- added copper zone on In2.Cu, net Net-(IC11-K)
- added copper zone on B.Cu, net Net-(IC12-K)
- added copper zone on F.Cu, net Net-(IC12-K)
- added copper zone on In1.Cu, net Net-(IC12-K)
- added copper zone on In2.Cu, net Net-(IC12-K)
- added copper zone on B.Cu, net Net-(IC13-K)
- added copper zone on F.Cu, net Net-(IC13-K)
- added copper zone on In1.Cu, net Net-(IC13-K)
- added copper zone on In2.Cu, net Net-(IC13-K)
- added copper zone on B.Cu, net Net-(IC6-K)
- added copper zone on F.Cu, net Net-(IC6-K)
- added copper zone on In1.Cu, net Net-(IC6-K)
- added copper zone on In2.Cu, net Net-(IC6-K)
- added copper zone on B.Cu, net Net-(IC7-K)
- added copper zone on F.Cu, net Net-(IC7-K)
- added copper zone on In1.Cu, net Net-(IC7-K)
- added copper zone on In2.Cu, net Net-(IC7-K)
- added copper zone on B.Cu, net Net-(IC8-K)
- added copper zone on F.Cu, net Net-(IC8-K)
- added copper zone on In1.Cu, net Net-(IC8-K)
- added copper zone on In2.Cu, net Net-(IC8-K)
- added copper zone on B.Cu, net Net-(IC9-K)
- added copper zone on F.Cu, net Net-(IC9-K)
- added copper zone on In1.Cu, net Net-(IC9-K)
- added copper zone on In2.Cu, net Net-(IC9-K)
Other:
- board text added: "+V"
- board text added: "0V"
- board text added: "ENC OUT 5V MAX"
- board text added: "FAB NOTE: the three circled vias sit inside J3 pads 9-11 (P31/P30/P29, 0.3 mm drill). Fill and cap them: IPC-4761 Type VII, epoxy filled and copper capped, planarized. All other vias: tented both sides."
- board text added: "OC: A B Z"
- board text added: "Rev v0.3"
- board text added: "VIN"
