File: Hardware/EdgeBoard/KiCad/MaD_Edge_Sheet2.kicad_sch (KiCad schematic)
At the start: 101 parts, among them IC1 ISO6742DWR, IC10 NSI50010YT1G, IC11 NSI50010YT1G, IC12 NSI50010YT1G, IC13 NSI50010YT1G, IC2 ISO6742DWR, IC3 UCC12040DVER, IC4 UCC12040DVER, IC5 ISO6731DWR, IC6 NSI50010YT1G, IC7 NSI50010YT1G, IC8 NSI50010YT1G, IC9 NSI50010YT1G, J10 ChargePump, J11 ESDUpper, J12 ESDLower, J13 ESDActive, J14 ENDUpper, J15 ENDLower, J16 Door, J17 GPI_3, J18 GPI_4, J19 NavKey, J4 436500321, J5 GPO_2, J6 GPO_1, J7 GPI_2, J8 GPI_1, J9 Force, U10 SN74LVC1G14DBV, U11 SN74LVC1G14DBV, U12 SN74LVC1G14DBV, U13 SN74LVC1G14DBV, U14 SN74LVC1G14DBV, U15 SN74LVC1G14DBV, U16 SN74LVC1G14DBV, U17 SN74LVC1G14DBV, U18 SN74LVC1G14DBV, U19 SN74LVC1G14DBV, U21 SN74LVC1G14DBV, U22 SN74LVC1G14DBV, U4 6N137, U5 VO2631, U6 VO2631, U7 VO2631, U8 VO2631, U9 SN74LVC1G14DBV

Commit message: DS2 and MaDEdge updates
Parts:
- J4: footprint Connector_Molex:Molex_Micro-Fit_3.0_43045-0618_2x03-1MP_P3.00mm_Vertical -> Connector_Molex:Molex_Micro-Fit_3.0_43045-0615_2x03_P3.00mm_Vertical
Connections:
- net IDOOR+: now also IC11.2 (A), J14.2 (Pin_2); no longer IC9.2 (A), J16.2 (Pin_2)
- net IDOOR-: now also J14.1 (Pin_1), U7.3 (C2); no longer J16.1 (Pin_1), U6.3 (C2)
- net IEND_U+: now also IC9.2 (A), J16.2 (Pin_2); no longer IC11.2 (A), J14.2 (Pin_2)
- net IEND_U-: now also J16.1 (Pin_1), U6.3 (C2); no longer J14.1 (Pin_1), U7.3 (C2)
- net IFG_RX: now also IC5.3 (INA), J9.2 (Pin_2); no longer IC5.5 (OUTC), J9.4 (Pin_4)
- net IFG_TX: now also IC5.5 (OUTC), J9.4 (Pin_4); no longer IC5.3 (INA), J9.2 (Pin_2)
- net RPI_RX: now also IC2.12 (INC), J4.3 (Pin_3); no longer IC2.14 (OUTA), J4.2 (Pin_2)
- net RPI_TX: now also IC2.14 (OUTA), J4.2 (Pin_2); no longer IC2.12 (INC), J4.3 (Pin_3)
