File: Hardware/EdgeBoard/KiCad/MaD_Edge_Sheet3.kicad_sch (KiCad schematic)
At the start: 60 parts, among them IC14 ISO7741FDWR, IC15 ISO6721BDR, IC16 ISO6740FDWR, J20 Encoder, J21 ServoCtrl, J23 ServoSerial, J25 ENC_PWR, Q1 MMBT3904, U24 AM26LS31CD, U25 AM26C32IDR, U27 SN74LVC1G14DBV, U28 SN74LVC1G14DBV, U29 SN74LVC1G14DBV, U30 SN74LVC1G14DBV, U31 SN74LVC1G14DBV, U32 SN74LVC1G14DBV, U33 SN74LVC1G14DBV, U34 SN74LVC1G14DBV

Commit message: docs(hardware): Edge carrier revision v0.3: marking and changelog
- Title blocks (three sheets and the PCB) and the silkscreen read v0.3.
- readme: the v0.3 changelog (each change, the finding, the datasheet
  cite), encoder jumper settings for RS-422, open-collector and push-pull
  encoders, the supported loop range, J1 as the host port, the P2-EC32MB
  pin facts, the J3 via-in-pad fab note, and the firmware/SIL follow-up.

Co-Authored-By: Claude Opus 5.5 <noreply@anthropic.com>
Other:
- company: (none) -> MaD
- title: (none) -> MaD Edge carrier: servo and encoder
Changed lines of the file:
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@@
 	(generator_version "9.0")
 	(paper "A4")
+	(title_block
+		(title "MaD Edge carrier: servo and encoder")
+		(date "2026-10-25")
+		(rev "v0.3")
+		(company "MaD")
+		(comment 1 "Revision v0.3: fixes from the SIL hardware findings; see Hardware/EdgeBoard/readme.md")
+	)
 	(junction
 		(at 34.29 48.26)

Commit message: fix(hardware): Q1 base resistor R24 43k -> 4.7k
With 43k from IC14 OUTC, Q1 gets about 77 uA of base current
((4.1 - 0.8) V / 43k at VOH min; SLLSEP4K 5.9 p.13). At the JSCJ MMBT3904's
minimum hFE of 100 (C20526 datasheet p.1) that limits the open-collector
enable to about 8 mA, and nothing in the repo records the drive's
enable-input current.

4.7k (UNI-ROYAL 0603WAF4701T5E, LCSC C23162, measured) gives 0.7-1.0 mA of
base current: a forced gain of 10-14 at 10 mA, near the datasheet's VCE(sat)
test ratio (IC/IB = 10 at 50 mA), and room for about 70 mA at hFE min
(inferred). OUTC then sources up to 1 mA into the base, inside the -4 mA
VOH test point (SLLSEP4K 5.9 p.13) and the +-15 mA absolute maximum
(5.1 p.6). The value is a judgement (see readme change 2).

Fields only; no connectivity change.

Co-Authored-By: Claude Opus 5.5 <noreply@anthropic.com>
Parts:
- R24: value 43K -> 4.7K; LCSC C23172 -> C23162; NOTES (none) -> Q1 base resistor: ~0.8 mA base drive so Q1 saturates at the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; manufacturer_part_number_1 0603WAF4302T5E -> 0603WAF4701T5E
Changed lines of the file:
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@@
 			)
 		)
-		(property "Value" "43K"
+		(property "Value" "4.7K"
 			(at 67.31 93.98 90)
 			(effects
@@
 			)
 		)
-		(property "LCSC" "C23172"
+		(property "LCSC" "C23162"
 			(at 69.85 91.44 0)
 			(effects
@@
 			)
 		)
-		(property "NOTES" ""
+		(property "NOTES" "Q1 base resistor: ~0.8 mA base drive so Q1 saturates at the drive enable current"
 			(at 69.85 91.44 0)
 			(effects
@@
 			)
 		)
-		(property "manufacturer_part_number_1" "0603WAF4302T5E"
+		(property "manufacturer_part_number_1" "0603WAF4701T5E"
 			(at 69.85 91.44 0)
 			(effects

Commit message: fix(hardware): BOM fields for F1, the 0.1 uF row, the shunts and J25
- F1: LCSC C7542932 is the LUTE 1206L020/30NR (LCSC product detail,
  measured): 0.20 A hold, 0.46 A trip, 30 V (LUTE 1206L datasheet, Revision
  2020, p.2). Manufacturer, trip current and datasheet link now say so.
- The 0.1 uF 0603 row (22 parts, C31 among them) orders LCSC C14663, the
  YAGEO CC0603KRX7R9BB104, 50 V X7R 0603 (LCSC product detail, measured).
  Its primary MPN was a Samsung 0402 part (CL05A104KA5NNNC) with a 6 V
  description. The MPN, manufacturer and description now match the ordered
  part; the DigiKey number that went with the Samsung MPN is cleared
  because it could not be checked.
- SH1-SH4: noted as hand-fit after assembly (no footprint, no CPL entry).
- IC14: note to check the ISO7741F top marking on receipt (SLLSEP4K
  package addendum p.38), since LCSC's parametric text for C485810 calls
  its fail-safe state high.
- J25: VIN is the encoder's own rated supply, 30 V max (F1), isolated from
  V_IN.

Fields only; no connectivity change.

Co-Authored-By: Claude Opus 5.5 <noreply@anthropic.com>
Parts:
- C24, C25, C26, C27, C28, C29, C31: DIGIKEY 1276-1043-1-ND -> (none); MANUFACTURER Samsung Electro-Mechanics -> YAGEO; Manufacturer_Part_Number CL05A104KA5NNNC -> CC0603KRX7R9BB104
- F1: MANUFACTURER Littelfuse -> LUTE; manufacturer_1 Littelfuse -> LUTE
- IC14: NOTES F suffix required: outputs default LOW with an open input or unpowered side 1 (SLLSEP4K Table 7-2). Do not fit a non-F part. -> F suffix required: outputs default LOW with an open input or unpowered side 1 (SLLSEP4K Table 7-2). Do not fit a non-F part. Check the top marking reads ISO7741F on receipt (SLLSEP4K package addendum).
- SH1: NOTES Shunt for JP1 (always fit): 1-2 = 5V drive enable, 2-3 = OC (sink) -> Shunt for JP1 (always fit): 1-2 = 5V drive enable, 2-3 = OC (sink). Hand-fit after assembly: no footprint, not in the CPL.
- SH2: NOTES Shunt for JP2 A_REF: fit only for an open-collector encoder -> Shunt for JP2 A_REF: fit only for an open-collector encoder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
- SH3: NOTES Shunt for JP3 B_REF: fit only for an open-collector encoder -> Shunt for JP3 B_REF: fit only for an open-collector encoder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
- SH4: NOTES Shunt for JP6 Z_REF: fit only for an open-collector encoder -> Shunt for JP6 Z_REF: fit only for an open-collector encoder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
Changed lines of the file:
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@@
 			)
 		)
-		(property "Description" "0.1uF 6V SMD"
+		(property "Description" "0.1uF 50V X7R 0603"
 			(at 34.29 50.8 0)
 			(effects
@@
 			)
 		)
-		(property "MANUFACTURER" "Samsung Electro-Mechanics"
+		(property "MANUFACTURER" "YAGEO"
 			(at 34.29 50.8 0)
 			(effects
@@
 			)
 		)
-		(property "Manufacturer_Part_Number" "CL05A104KA5NNNC"
+		(property "Manufacturer_Part_Number" "CC0603KRX7R9BB104"
 			(at 34.29 50.8 0)
 			(effects
@@
 			)
 		)
-		(property "DIGIKEY" "1276-1043-1-ND"
+		(property "DIGIKEY" ""
 			(at 34.29 50.8 0)
 			(effects
@@
 			)
 		)
-		(property "Description" "0.1uF 6V SMD"
+		(property "Description" "0.1uF 50V X7R 0603"
 			(at 74.93 27.94 0)
 			(effects
@@
 			)
 		)
-		(property "MANUFACTURER" "Samsung Electro-Mechanics"
+		(property "MANUFACTURER" "YAGEO"
 			(at 74.93 27.94 0)
 			(effects
@@
 			)
 		)
-		(property "Manufacturer_Part_Number" "CL05A104KA5NNNC"
+		(property "Manufacturer_Part_Number" "CC0603KRX7R9BB104"
 			(at 74.93 27.94 0)
 			(effects
@@
 			)
 		)
-		(property "DIGIKEY" "1276-1043-1-ND"
+		(property "DIGIKEY" ""
 			(at 74.93 27.94 0)
 			(effects
@@
 			)
 		)
-		(property "Description" "0.1uF 6V SMD"
+		(property "Description" "0.1uF 50V X7R 0603"
 			(at 85.09 49.53 0)
 			(effects
@@
 			)
 		)
-		(property "MANUFACTURER" "Samsung Electro-Mechanics"
+		(property "MANUFACTURER" "YAGEO"
 			(at 85.09 49.53 0)
 			(effects
@@
 			)
 		)
-		(property "Manufacturer_Part_Number" "CL05A104KA5NNNC"
+		(property "Manufacturer_Part_Number" "CC0603KRX7R9BB104"
 			(at 85.09 49.53 0)
 			(effects
@@
 			)
 		)
-		(property "DIGIKEY" "1276-1043-1-ND"
+		(property "DIGIKEY" ""
 			(at 85.09 49.53 0)
 			(effects
@@
 			)
 		)
-		(property "Description" "0.1uF 6V SMD"
+		(property "Description" "0.1uF 50V X7R 0603"
 			(at 125.73 22.86 0)
 			(effects
@@
 			)
 		)
-		(property "MANUFACTURER" "Samsung Electro-Mechanics"
+		(property "MANUFACTURER" "YAGEO"
 			(at 125.73 22.86 0)
 			(effects
@@
 			)
 		)
-		(property "Manufacturer_Part_Number" "CL05A104KA5NNNC"
+		(property "Manufacturer_Part_Number" "CC0603KRX7R9BB104"
 			(at 125.73 22.86 0)
 			(effects
@@
 			)
 		)
-		(property "DIGIKEY" "1276-1043-1-ND"
+		(property "DIGIKEY" ""
 			(at 125.73 22.86 0)
 			(effects
@@
 			)
 		)
-		(property "Description" "0.1uF 6V SMD"
+		(property "Description" "0.1uF 50V X7R 0603"
 			(at 35.56 124.46 0)
 			(effects
@@
 			)
 		)
-		(property "MANUFACTURER" "Samsung Electro-Mechanics"
+		(property "MANUFACTURER" "YAGEO"
 			(at 35.56 124.46 0)
 			(effects
@@
 			)
 		)
-		(property "Manufacturer_Part_Number" "CL05A104KA5NNNC"
+		(property "Manufacturer_Part_Number" "CC0603KRX7R9BB104"
 			(at 35.56 124.46 0)
 			(effects
@@
 			)
 		)
-		(property "DIGIKEY" "1276-1043-1-ND"
+		(property "DIGIKEY" ""
 			(at 35.56 124.46 0)
 			(effects
@@
 			)
 		)
-		(property "Description" "0.1uF 6V SMD"
+		(property "Description" "0.1uF 50V X7R 0603"
 			(at 76.2 124.46 0)
 			(effects
@@
 			)
 		)
-		(property "MANUFACTURER" "Samsung Electro-Mechanics"
+		(property "MANUFACTURER" "YAGEO"
 			(at 76.2 124.46 0)
 			(effects
@@
 			)
 		)
-		(property "Manufacturer_Part_Number" "CL05A104KA5NNNC"
+		(property "Manufacturer_Part_Number" "CC0603KRX7R9BB104"
 			(at 76.2 124.46 0)
 			(effects
@@
 			)
 		)
-		(property "DIGIKEY" "1276-1043-1-ND"
+		(property "DIGIKEY" ""
 			(at 76.2 124.46 0)
 			(effects
@@
 			)
 		)
-		(property "NOTES" "F suffix required: outputs default LOW with an open input or unpowered side 1 (SLLSEP4K Table 7-2). Do not fit a non-F part."
+		(property "NOTES" "F suffix required: outputs default LOW with an open input or unpowered side 1 (SLLSEP4K Table 7-2). Do not fit a non-F part. Check the top marking reads ISO7741F on receipt (SLLSEP4K package addendum)."
 			(at 39.37 50.8 0)
 			(effects
@@
 			)
 		)
-		(property "Description" "0.1uF 6V SMD"
+		(property "Description" "0.1uF 50V X7R 0603"
 			(at 209.55 120.65 0)
 			(effects
@@
 			)
 		)
-		(property "MANUFACTURER" "Samsung Electro-Mechanics"
+		(property "MANUFACTURER" "YAGEO"
 			(at 209.55 120.65 0)
 			(effects
@@
 			)
 		)
-		(property "Manufacturer_Part_Number" "CL05A104KA5NNNC"
+		(property "Manufacturer_Part_Number" "CC0603KRX7R9BB104"
 			(at 209.55 120.65 0)
 			(effects
@@
 			)
 		)
-		(property "DIGIKEY" "1276-1043-1-ND"
+		(property "DIGIKEY" ""
 			(at 209.55 120.65 0)
 			(effects
@@
 			)
 		)
-		(property "Description" "Encoder supply pass-through: 1 VIN (7-24 V in), 2 ENC+ (fused, to encoder V+), 3 0V (EN_GND)"
+		(property "Description" "Encoder supply pass-through: 1 VIN (the encoder's rated supply, 30 V max, isolated from V_IN), 2 +V (fused, to encoder V+), 3 0V (EN_GND)"
 			(at 273.05 115.57 0)
 			(effects
@@
 			)
 		)
-		(property "Datasheet" "https://www.littelfuse.com/assetdocs/littelfuse-ptc-1206l-datasheet"
+		(property "Datasheet" "https://www.lcsc.com/datasheet/C7542932.pdf"
 			(at 246.38 115.57 0)
 			(effects
@@
 			)
 		)
-		(property "Description" "PTC, 0.20 A hold, 0.42 A trip, 30 V, 1206 (encoder supply)"
+		(property "Description" "PTC, 0.20 A hold, 0.46 A trip, 30 V, 1206 (encoder supply)"
 			(at 246.38 115.57 0)
 			(effects
@@
 			)
 		)
-		(property "MANUFACTURER" "Littelfuse"
+		(property "MANUFACTURER" "LUTE"
 			(at 246.38 115.57 0)
 			(effects
@@
 			)
 		)
-		(property "manufacturer_1" "Littelfuse"
+		(property "manufacturer_1" "LUTE"
 			(at 246.38 115.57 0)
 			(effects
@@
 			)
 		)
-		(property "NOTES" "Shunt for JP1 (always fit): 1-2 = 5V drive enable, 2-3 = OC (sink)"
+		(property "NOTES" "Shunt for JP1 (always fit): 1-2 = 5V drive enable, 2-3 = OC (sink). Hand-fit after assembly: no footprint, not in the CPL."
 			(at 175.26 140.97 0)
 			(effects
@@
 			)
 		)
-		(property "NOTES" "Shunt for JP2 A_REF: fit only for an open-collector encoder"
+		(property "NOTES" "Shunt for JP2 A_REF: fit only for an open-collector encoder. Hand-fit after assembly: no footprint, not in the CPL."
 			(at 190.5 140.97 0)
 			(effects
@@
 			)
 		)
-		(property "NOTES" "Shunt for JP3 B_REF: fit only for an open-collector encoder"
+		(property "NOTES" "Shunt for JP3 B_REF: fit only for an open-collector encoder. Hand-fit after assembly: no footprint, not in the CPL."
 			(at 205.74 140.97 0)
 			(effects
@@
 			)
 		)
-		(property "NOTES" "Shunt for JP6 Z_REF: fit only for an open-collector encoder"
+		(property "NOTES" "Shunt for JP6 Z_REF: fit only for an open-collector encoder. Hand-fit after assembly: no footprint, not in the CPL."
 			(at 220.98 140.97 0)
 			(effects
