File: Hardware/EdgeBoard/KiCad/MaD_Edge_Sheet3.kicad_sch (KiCad schematic)
At the start: 46 parts, among them IC14 ISO6741DWR, IC15 ISO6721BDR, IC16 ISO6740FDWR, J20 Encoder, J21 ServoCtrl, J23 ServoSerial, Q1 NPN, U24 AM26LS31CD, U25 AM26LV32IDR, U27 SN74LVC1G14DBV, U28 SN74LVC1G14DBV, U29 SN74LVC1G14DBV, U30 SN74LVC1G14DBV, U31 SN74LVC1G14DBV, U32 SN74LVC1G14DBV, U33 SN74LVC1G14DBV, U34 SN74LVC1G14DBV

Commit message: Edge carrier revision: fixes from the SIL hardware findings (#309)
* fix(hardware): servo enable off at power-up: IC14 ISO7741FDWR and a P6 pull-down

Finding SRV-F6. Nothing pulls P6 (servo enable request), and the fitted
non-F IC14 outputs high from an open or unpowered input, so the drive
enable is on through reset, boot and flashing.

- IC14 becomes ISO7741FDWR (LCSC C485810): same pinout (TI SLLSEP4K
  Table 4-1 p.5); with the F suffix an open input or an unpowered side 1
  gives a low output (Table 7-2 p.29). Value, MPN, LCSC and notes updated.
- R39, 10 k (0603WAF1002T5E, C25804) from P6 to GND. On the PCB it sits
  by IC14 and joins the P6 trace at U29 through two 0.6 mm vias and B.Cu.
- STEP/DIR (P8/P7) now also rest low when undriven.

Co-Authored-By: Claude Opus 5.5 <noreply@anthropic.com>

* fix(hardware): Q1 drawn and laid out as the fitted SOT-23 MMBT3904

Finding SRV-F8-Q1. Q1 used the TO-92 2N3904 symbol (1 E, 2 B, 3 C) but
the part fitted is a SOT-23 MMBT3904 (1 B, 2 E, 3 C; JSCJ datasheet,
LCSC C20526, p.1), so JP1's open-collector position could never enable
the drive.

- Symbol Transistor_BJT:MMBT3904, footprint Package_TO_SOT_SMD:SOT-23.
- PCB: Q1 rotated -90 so base faces R24; base to R24, emitter to a new
  EN_GND via, collector to JP1 pin 3. The old emitter trace and via go.

Co-Authored-By: Claude Opus 5.5 <noreply@anthropic.com>

* fix(hardware): U25 AM26C32IDR (5 V receiver) with its own 0.1 uF

Finding ENC-F3. U25 (AM26LV32IDR, 3.0-3.6 V, TI SLLS202H 6.3) runs from
the 5 V SC_5V rail.

- U25 becomes AM26C32IDR (LCSC C36693): pin-identical (TI SLLS104M
  Table 4-1 p.3), VCC 4.5-5.5 V (5.3 p.4), VOH >= 3.8 V at -6 mA (5.6
  p.5), above IC16's 0.7 x VCC1 input threshold. KiCad has no AM26C32
  symbol; the AM26LV32xD symbol stays.
- C30, 0.1 uF 0402 (CL05B104KO5NNNC, C1525) from U25.16 to EN_GND,
  beside the pin. 0402 is the size that fits between JP2 and U25.

Co-Authored-By: Claude Opus 5.5 <noreply@anthropic.com>

* fix(hardware): U25 alw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
Parts:
- removed JP4: Z_GND, Connector_PinHeader_2.54mm:PinHeader_1x02_P2.54mm_Vertical, symbol Jumper:Jumper_2_Open
- added C30: 0.1uF, Capacitor_SMD:C_0402_1005Metric, symbol Device:C_Small
- added C31: 0.1uF, Capacitor_SMD:C_0603_1608Metric, symbol Device:C_Small
- added F1: 0.2A/30V, Fuse:Fuse_1206_3216Metric, symbol Device:Polyfuse_Small
- added J25: ENC_PWR, Connector_PinHeader_2.54mm:PinHeader_1x03_P2.54mm_Vertical, symbol Connector_Generic:Conn_01x03
- added JP6: Z_REF, Connector_PinHeader_2.54mm:PinHeader_1x02_P2.54mm_Vertical, symbol Jumper:Jumper_2_Open
- added R39: 10K, Resistor_SMD:R_0603_1608Metric, symbol Device:R_Small
- added R40, R41, R42, R43, R44: 2.2K, Resistor_SMD:R_0603_1608Metric, symbol Device:R_Small
- added SH1, SH2, SH3, SH4: Shunt 2.54mm, symbol Mechanical:Housing
- C24, C25, C26, C27, C28, C29: DIGIKEY 1276-1043-1-ND -> (none); MANUFACTURER Samsung Electro-Mechanics -> YAGEO; Manufacturer_Part_Number CL05A104KA5NNNC -> CC0603KRX7R9BB104
- IC14: value ISO6741DWR -> ISO7741FDWR; DIGIKEY 296-ISO6741DWRCT-ND -> (none); LCSC C571196 -> C485810; Manufacturer_Part_Number ISO6741DWR -> ISO7741FDWR; NOTES Pin Compatible with ISO77xx -> F suffix required: outputs default LOW with an open input o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; Qty Bought 3 - lcsc -> (none); manufacturer_part_number_1 ISO6741DWR or ISO7741DWR -> ISO7741FDWR
- JP2: value A_GND -> A_REF; NOTES (none) -> Shunt only for a single-ended open-collector encoder; OPEN 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
- JP3: value B_GND -> B_REF; NOTES (none) -> Shunt only for a single-ended open-collector encoder; OPEN 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
- JP5: value ZI_GND -> ZI_REF; NOTES (none) -> Shunt only for a single-ended push-pull (TTL) ZI signal; OP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
- Q1: value NPN -> MMBT3904; footprint Package_TO_SOT_SMD:TSOT-23 -> Package_TO_SOT_SMD:SOT-23; symbol Transistor_BJT:2N3904 -> Transistor_BJT:MMBT3904; NOTES (none) -> SOT-23 pinout 1 B, 2 E, 3 C (JSCJ MMBT3904 datasheet p.1)
- R24: value 43K -> 4.7K; LCSC C23172 -> C23162; NOTES (none) -> Q1 base resistor: ~0.8 mA base drive so Q1 saturates at the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; manufacturer_part_number_1 0603WAF4302T5E -> 0603WAF4701T5E
- U25: value AM26LV32IDR -> AM26C32IDR; LCSC C524786 -> C36693; Manufacturer_Part_Number AM26LV32IDR -> AM26C32IDR; NOTES (none) -> Must be a 5 V receiver (AM26C32, VCC 4.5-5.5 V, VOH >= 3.8 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; Qty Bought 3 lcsc -> (none); manufacturer_part_number_1 AM26LV32IDR -> AM26C32IDR
Connections:
- net A+: now also R40.2
- net B+: now also R41.2
- net EN_GND: now also Q1.2 (E), U25.12 (~{G}), C30.2, C31.2, J25.3 (Pin_3), R44.2; no longer JP2.2 (B), JP3.2 (B), JP5.2 (B), Q1.1 (E)
- net GND: now also R39.2
- net P6: now also R39.1
- net SC_5V: now also U25.4 (G), C30.1, R40.1, R41.1, R42.1, R43.1
- net Z+: now also U25.14 (4A), R42.2; no longer U25.4 (G)
- net Z-: now also U25.15 (4B), JP6.1 (A); no longer U25.12 (~{G})
- net at R24.2: now also Q1.1 (B); no longer Q1.2 (B)
- new net ENC_REF: C31.1, JP2.2 (B), JP3.2 (B), JP5.2 (B), JP6.2 (B), R43.2, R44.1
- new net ENC_V+: F1.2, J25.2 (Pin_2)
- new net ENC_VIN: F1.1, J25.1 (Pin_1)
- no-connect marks 11 -> 9
Other:
- note added: "Encoder input (v0.3): R40-R42 pull A+/B+/Z+ up for an open-collector A/B/Z encoder. JP2/JP3/JP6/JP5 tie A-/B-/Z-/ZI- to ENC_REF (SC_5V/2: R43/R44, C31). Open-collector (NPN) encoder on A+/B+/Z+: fit JP2, JP3, JP6. RS-422 line driver: all four OPEN. J25: encoder supply pass-through (1 VIN, 2 ENC+ via F1, 3 0V). U25 is a 5 V AM26C32."
- note added: "R39 holds P6 low: servo enable off through reset, boot and flashing. IC14 is an F part: outputs default low if side 1 is unpowered."
- company: (none) -> MaD
- title: (none) -> MaD Edge carrier: servo and encoder
