File: Hardware/EdgeBoard/KiCad/MaD_Edge.kicad_sch (KiCad schematic)
At the start: 21 parts, among them J1 Debug, J2 Main_Power, J22 GPIO_EXT_1, J24 GPIO_EXT_2, J3 P2_EDGE_MODULE_SOCKET, SW1 RESET, U1 XL1509-5V, U2 XL1509-3.3V, U3 APM4953

Commit message: Edge carrier revision: fixes from the SIL hardware findings (#309)
* fix(hardware): servo enable off at power-up: IC14 ISO7741FDWR and a P6 pull-down

Finding SRV-F6. Nothing pulls P6 (servo enable request), and the fitted
non-F IC14 outputs high from an open or unpowered input, so the drive
enable is on through reset, boot and flashing.

- IC14 becomes ISO7741FDWR (LCSC C485810): same pinout (TI SLLSEP4K
  Table 4-1 p.5); with the F suffix an open input or an unpowered side 1
  gives a low output (Table 7-2 p.29). Value, MPN, LCSC and notes updated.
- R39, 10 k (0603WAF1002T5E, C25804) from P6 to GND. On the PCB it sits
  by IC14 and joins the P6 trace at U29 through two 0.6 mm vias and B.Cu.
- STEP/DIR (P8/P7) now also rest low when undriven.

Co-Authored-By: Claude Opus 5.5 <noreply@anthropic.com>

* fix(hardware): Q1 drawn and laid out as the fitted SOT-23 MMBT3904

Finding SRV-F8-Q1. Q1 used the TO-92 2N3904 symbol (1 E, 2 B, 3 C) but
the part fitted is a SOT-23 MMBT3904 (1 B, 2 E, 3 C; JSCJ datasheet,
LCSC C20526, p.1), so JP1's open-collector position could never enable
the drive.

- Symbol Transistor_BJT:MMBT3904, footprint Package_TO_SOT_SMD:SOT-23.
- PCB: Q1 rotated -90 so base faces R24; base to R24, emitter to a new
  EN_GND via, collector to JP1 pin 3. The old emitter trace and via go.

Co-Authored-By: Claude Opus 5.5 <noreply@anthropic.com>

* fix(hardware): U25 AM26C32IDR (5 V receiver) with its own 0.1 uF

Finding ENC-F3. U25 (AM26LV32IDR, 3.0-3.6 V, TI SLLS202H 6.3) runs from
the 5 V SC_5V rail.

- U25 becomes AM26C32IDR (LCSC C36693): pin-identical (TI SLLS104M
  Table 4-1 p.3), VCC 4.5-5.5 V (5.3 p.4), VOH >= 3.8 V at -6 mA (5.6
  p.5), above IC16's 0.7 x VCC1 input threshold. KiCad has no AM26C32
  symbol; the AM26LV32xD symbol stays.
- C30, 0.1 uF 0402 (CL05B104KO5NNNC, C1525) from U25.16 to EN_GND,
  beside the pin. 0402 is the size that fits between JP2 and U25.

Co-Authored-By: Claude Opus 5.5 <noreply@anthropic.com>

* fix(hardware): U25 alw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
Other:
- company: (none) -> MaD
- title: (none) -> MaD Edge carrier
Changed lines of the file:
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@@
 	(generator_version "9.0")
 	(paper "A4")
+	(title_block
+		(title "MaD Edge carrier")
+		(date "2026-10-25")
+		(rev "v0.3")
+		(company "MaD")
+		(comment 1 "Revision v0.3: fixes from the SIL hardware findings; see Hardware/EdgeBoard/readme.md")
+	)
 	(text "Debug/Programming"
 		(exclude_from_sim no)
