File: Hardware/DS2Addon/KICAD/DS2_Addon.kicad_pcb (KiCad board)
At the start: 2 copper layers, 47 x 25.4 mm, 34 parts, among them J1 MCU, J2 Analog1, J3 Conn_01x03, J4 Reference, J5 Analog2, U1 ADS122U04

Commit message: fix(hardware): add 10k pull-up on ADS122U04 ~RESET (DS2 Addon)
U1 pin 3 (~RESET) was left floating -- the ~{RESET} net contained only
U1.3, no pull-up or connector. Per SBAS752B (Unused Inputs and Outputs)
unused digital inputs must be tied to DVDD or DGND; on two physical
boards the chip did not respond to any UART command until ~RESET was
manually tied to 3.3 V.

- Add R10 (10k, 0805) from ~RESET to +3V3 in the schematic
- Place R10 east of U1 and route it: pad 3 was boxed in on F.Cu, so the
  U1 pad 4 GND stub is rerouted east to a new via (still in the B.Cu
  GND zone), and +3V3 crosses on B.Cu with two vias onto the existing
  DVDD trace; zones refilled
- Document bench testing in the readme (J2 AVDD/AGND straps, JP1/JP2
  jumpers, RX->P2 / TX->P0 @ 115200, pre-R10 bodge)

ERC/DRC (kicad-cli 9.0.6, --severity-all, --schematic-parity): no new
violations; the floating-~RESET ERC findings are resolved and the zone
refill fixed 3 pre-existing DRC violations (2 copper slivers, 1 starved
thermal).

Co-Authored-By: Claude Fable 5 <noreply@anthropic.com>
Parts:
- added R10: 10k, Resistor_SMD:R_0805_2012Metric, F.Cu at (143.8, 86.5)
Routing:
- net +3V3: track 11.9 -> 22.0 mm, vias 0 -> 2
- net GND: track 7.18 -> 12.7 mm
- net ~{RESET}: track 0.00 -> 3.38 mm
Changed lines of the file:
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@@
 		(embedded_fonts no)
 	)
+	(footprint "Resistor_SMD:R_0805_2012Metric"
+		(layer "F.Cu")
+		(at 143.8 86.55)
+		(descr "Resistor SMD 0805 (2012 Metric), square (rectangular) end terminal, IPC-7351 nominal, (Body size source: IPC-SM-782 page 72, https://www.pcb-3d.com/wordpress/wp-content/uploads/ipc-sm-782a_amendment_1_and_2.pdf), generated with kicad-footprint-generator")
+		(tags "resistor")
+		(property "Reference" "R10"
+			(at 0 -1.65 0)
+			(layer "F.SilkS")
+			(hide yes)
+			(effects
+				(font
+					(size 1 1)
+					(thickness 0.15)
+				)
+			)
+		)
+		(property "Value" "10k"
+			(at 0 1.65 0)
+			(layer "F.Fab")
+			(effects
+				(font
+					(size 1 1)
+					(thickness 0.15)
+				)
+			)
+		)
+		(property "Datasheet" ""
+			(at 0 0 0)
+			(layer "F.Fab")
+			(hide yes)
+			(effects
+				(font
+					(size 1.27 1.27)
+					(thickness 0.15)
+				)
+			)
+		)
+		(property "Description" ""
+			(at 0 0 0)
+			(layer "F.Fab")
+			(hide yes)
+			(effects
+				(font
+					(size 1.27 1.27)
+					(thickness 0.15)
+				)
+			)
+		)
+		(attr smd)
+		(fp_line
+			(start -0.227064 -0.735)
+			(end 0.227064 -0.735)
+			(stroke
+				(width 0.12)
+				(type solid)
+			)
+			(layer "F.SilkS")
+		)
+		(fp_line
+			(start -0.227064 0.735)
+			(end 0.227064 0.735)
+			(stroke
+				(width 0.12)
+				(type solid)
+			)
+			(layer "F.SilkS")
+		)
+		(fp_line
+			(start -1.68 -0.95)
+			(end 1.68 -0.95)
+			(stroke
+				(width 0.05)
+				(type solid)
+			)
+			(layer "F.CrtYd")
+		)
+		(fp_line
+			(start -1.68 0.95)
+			(end -1.68 -0.95)
+			(stroke
+				(width 0.05)
+				(type solid)
+			)
+			(layer "F.CrtYd")
+		)
+		(fp_line
+			(start 1.68 -0.95)
+			(end 1.68 0.95)
+			(stroke
+				(width 0.05)
+				(type solid)
+			)
+			(layer "F.CrtYd")
+		)
+		(fp_line
+			(start 1.68 0.95)
+			(end -1.68 0.95)
+			(stroke
+				(width 0.05)
+				(type solid)
+			)
+			(layer "F.CrtYd")
+		)
+		(fp_line
+			(start -1 -0.625)
+			(end 1 -0.625)
+			(stroke
+				(width 0.1)
+				(type solid)
+			)
+			(layer "F.Fab")
+		)
+		(fp_line
+			(start -1 0.625)
+			(end -1 -0.625)
+			(stroke
+				(width 0.1)
+				(type solid)
+			)
+			(layer "F.Fab")
+		)
+		(fp_line
+			(start 1 -0.625)
+			(end 1 0.625)
+			(stroke
+				(width 0.1)
+				(type solid)
+			)
+			(layer "F.Fab")
+		)
+		(fp_line
+			(start 1 0.625)
+			(end -1 0.625)
+			(stroke
+				(width 0.1)
+				(type solid)
+			)
+			(layer "F.Fab")
+		)
+		(fp_text user "${REFERENCE}"
+			(at 0 0 0)
+			(layer "F.Fab")
+			(effects
+				(font
+					(size 0.5 0.5)
+					(thickness 0.08)
+				)
+			)
+		)
+		(pad "1" smd roundrect
+			(at -0.9125 0)
+			(size 1.025 1.4)
+			(layers "F.Cu" "F.Mask" "F.Paste")
+			(roundrect_rratio 0.243902)
+			(net 24 "~{RESET}")
+		)
+		(pad "2" smd roundrect
+			(at 0.9125 0)
+			(size 1.025 1.4)
+			(layers "F.Cu" "F.Mask" "F.Paste")
+			(roundrect_rratio 0.243902)
+			(net 4 "+3V3")
+		)
+		(embedded_fonts no)
+		(model "${KICAD9_3DMODEL_DIR}/Resistor_SMD.3dshapes/R_0805_2012Metric.step"
+			(offset
+				(xyz 0 0 0)
+			)
+			(scale
+				(xyz 1 1 1)
+			)
+			(rotate
+				(xyz 0 0 0)
+			)
+		)
+	)
 	(footprint "DS2_Addon:LOGO"
 		(layer "B.Cu")
@@
 	)
 	(segment
+		(start 144.7125 86.55)
+		(end 144.7125 87.6)
+		(width 0.25)
+		(layer "F.Cu")
+		(net 4)
+	)
+	(segment
 		(start 135.89 89.535)
 		(end 133.985 89.535)
@@
 		(net 4)
 	)
+	(via
+		(at 144.7125 87.6)
+		(size 0.8)
+		(drill 0.4)
+		(layers "F.Cu" "B.Cu")
+		(net 4)
+	)
+	(via
+		(at 135.89 88.2)
+		(size 0.8)
+		(drill 0.4)
+		(layers "F.Cu" "B.Cu")
+		(net 4)
+	)
+	(segment
+		(start 136.49 87.6)
+		(end 135.89 88.2)
+		(width 0.25)
+		(layer "B.Cu")
+		(net 4)
+	)
+	(segment
+		(start 144.7125 87.6)
+		(end 136.49 87.6)
+		(width 0.25)
+		(layer "B.Cu")
+		(net 4)
+	)
 	(segment
 		(start 139.705 85.415)
@@
 	(segment
 		(start 140.393558 85.415)
-		(end 141.592558 86.614)
+		(end 145.6 85.415)
 		(width 0.25)
 		(layer "F.Cu")
@@
 	)
 	(segment
-		(start 138.811 89.535)
-		(end 138.938 89.662)
+		(start 145.6 85.415)
+		(end 146.5 86.315)
 		(width 0.25)
 		(layer "F.Cu")
@@
 	)
 	(segment
-		(start 141.592558 86.614)
-		(end 141.732 86.614)
+		(start 146.5 86.315)
+		(end 146.5 87.2)
+		(width 0.25)
+		(layer "F.Cu")
+		(net 5)
+	)
+	(segment
+		(start 138.811 89.535)
+		(end 138.938 89.662)
 		(width 0.25)
 		(layer "F.Cu")
@@
 	)
 	(via
-		(at 141.732 86.614)
+		(at 146.5 87.2)
 		(size 0.8)
 		(drill 0.4)
@@
 	)
 	(segment
+		(start 139.705 86.065)
+		(end 142.4 86.065)
+		(width 0.25)
+		(layer "F.Cu")
+		(net 24)
+	)
+	(segment
+		(start 142.4 86.065)
+		(end 142.8875 86.55)
+		(width 0.25)
+		(layer "F.Cu")
+		(net 24)
+	)
+	(segment
