File: Hardware/DS2Addon/KICAD/DS2_Addon.kicad_sch (KiCad schematic)
At the start: 31 parts, among them J1 MCU, J2 Analog1, J3 Conn_01x03, J4 Reference, J5 Analog2, U1 ADS122U04

Commit message: fix(hardware): add 10k pull-up on ADS122U04 ~RESET (DS2 Addon)
U1 pin 3 (~RESET) was left floating -- the ~{RESET} net contained only
U1.3, no pull-up or connector. Per SBAS752B (Unused Inputs and Outputs)
unused digital inputs must be tied to DVDD or DGND; on two physical
boards the chip did not respond to any UART command until ~RESET was
manually tied to 3.3 V.

- Add R10 (10k, 0805) from ~RESET to +3V3 in the schematic
- Place R10 east of U1 and route it: pad 3 was boxed in on F.Cu, so the
  U1 pad 4 GND stub is rerouted east to a new via (still in the B.Cu
  GND zone), and +3V3 crosses on B.Cu with two vias onto the existing
  DVDD trace; zones refilled
- Document bench testing in the readme (J2 AVDD/AGND straps, JP1/JP2
  jumpers, RX->P2 / TX->P0 @ 115200, pre-R10 bodge)

ERC/DRC (kicad-cli 9.0.6, --severity-all, --schematic-parity): no new
violations; the floating-~RESET ERC findings are resolved and the zone
refill fixed 3 pre-existing DRC violations (2 copper slivers, 1 starved
thermal).

Co-Authored-By: Claude Fable 5 <noreply@anthropic.com>
Parts:
- added R10: 10k, Resistor_SMD:R_0805_2012Metric, symbol Device:R_Small
Connections:
- net +3V3: now also R10.2
- net ~{RESET}: now also R10.1
Changed lines of the file:
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@@
+    )
+  )
+  (global_label "~{RESET}" (shape input) (at 109.22 81.28 270)
+    (effects (font (size 1.27 1.27)) (justify right))
+    (property "Intersheetrefs" "${INTERSHEET_REFS}" (at 109.22 81.28 0)
+      (effects (font (size 1.27 1.27)) hide)
     )
   )
@@
         )
       )
+    )
+  )
+  (symbol (lib_id "Device:R_Small") (at 109.22 78.74 180) (unit 1)
+    (in_bom yes) (on_board yes) (dnp no)
+    (property "Reference" "R10" (at 107.315 78.74 90)
+      (effects (font (size 1.27 1.27)))
+    )
+    (property "Value" "10k" (at 111.125 78.74 90)
+      (effects (font (size 1.27 1.27)))
+    )
+    (property "Footprint" "Resistor_SMD:R_0805_2012Metric" (at 109.22 78.74 0)
+      (effects (font (size 1.27 1.27)) hide)
+    )
+    (property "Datasheet" "~" (at 109.22 78.74 0)
+      (effects (font (size 1.27 1.27)) hide)
+    )
+    (property "LCSC" "~" (at 109.22 78.74 0)
+      (effects (font (size 1.27 1.27)) hide)
+    )
+    (pin "1")
+    (pin "2")
+    (instances
+      (project "DS2_Addon"
+        (path "/c7b55e36-b373-4bc4-ba40-ef53ef8dff09"
+          (reference "R10") (unit 1)
+        )
+      )
+    )
+  )
+  (symbol (lib_id "power:+3V3") (at 109.22 76.2 0) (unit 1)
+    (in_bom yes) (on_board yes) (dnp no)
+    (property "Reference" "#PWR0118" (at 109.22 80.01 0)
+      (effects (font (size 1.27 1.27)) hide)
+    )
+    (property "Value" "+3V3" (at 109.601 71.8058 0)
+      (effects (font (size 1.27 1.27)))
+    )
+    (property "Footprint" "" (at 109.22 76.2 0)
+      (effects (font (size 1.27 1.27)) hide)
+    )
+    (property "Datasheet" "" (at 109.22 76.2 0)
+      (effects (font (size 1.27 1.27)) hide)
+    )
+    (pin "1")
+    (instances
+      (project "DS2_Addon"
+        (path "/c7b55e36-b373-4bc4-ba40-ef53ef8dff09"
+          (reference "#PWR0118") (unit 1)
+        )
+      )
